Commit message: 阶段修改

File: data/cameras/camera3d.urdf (robot description, URDF)
Before this commit: robot canera3d, 2 links, 1 joints
Links:
- link base: geometry collision box size=0.1 0.1 2.5; visual mesh filename=camera3d/camera.obj scale=1 1 1

File: data/end_effectors/nozzle/nozzle.urdf (robot description, URDF)
Before this commit: robot universal_robot, 3 links, 2 joints
Links:
- removed link placeholder
- added link ee_link; visual box size=0.01 0.01 0.01
- link ee: geometry visual mesh filename=link1.obj scale=1.2 1.2 2
Joints:
- joint joint_ee: origin xyz=0 0.065 0 rpy=0 0 0 -> xyz=0 0.07 0 rpy=1.57 0 0
