Commit message: 阶段提交

File: data/end_effectors/motoman/motoman.urdf (robot description, URDF)
Before this commit: robot universal_robot, 3 links, 2 joints
Joints:
- joint joint_ee: origin xyz=0.12 0 0.25 rpy=0 0.0 0 -> xyz=0.12 0 0.25 rpy=0 3.14 1.57

Commit message: 阶段提交

File: data/end_effectors/motoman/motoman.urdf (robot description, URDF)
Before this commit: robot universal_robot, 3 links, 2 joints
Links:
- link ee: mass None -> .01
Joints:
- joint joint_ee: origin xyz=0.12 0 0.25 rpy=0 3.14 1.57 -> xyz=0.12 0 0.24 rpy=0 0 0
