Commit message: 阶段提交

File: data/robots/franka_panda/franka_panda.urdf (robot description, URDF)
Before this commit: robot panda, 13 links, 12 joints
Links:
- removed link panda_grasptarget
- removed link panda_hand
- removed link panda_leftfinger
- removed link panda_link8
- removed link panda_rightfinger
- added link placeholder; visual box size=0.01 0.01 0.01
- link panda_link0: geometry collision mesh filename=collision/link0.obj; visual mesh filename=collision/link0.obj
- link panda_link1: geometry collision mesh filename=collision/link1.obj; visual mesh filename=visual/link1.obj
- link panda_link2: geometry collision mesh filename=collision/link2.obj; visual mesh filename=visual/link2.obj
- link panda_link3: geometry collision mesh filename=collision/link3.obj; visual mesh filename=visual/link3.obj
- link panda_link4: geometry collision mesh filename=collision/link4.obj; visual mesh filename=visual/link4.obj
- link panda_link5: geometry collision mesh filename=collision/link5.obj; visual mesh filename=visual/link5.obj
- link panda_link6: geometry collision mesh filename=collision/link6.obj; visual mesh filename=visual/link6.obj
- link panda_link7: geometry collision mesh filename=collision/link7.obj; visual mesh filename=collision/link7.obj
Joints:
- removed joint panda_finger_joint1
- removed joint panda_finger_joint2
- removed joint panda_grasptarget_hand
- removed joint panda_hand_joint
- joint panda_joint8: child panda_link8 -> placeholder
