Commit message: 阶段提交

File: data/objects/box/box.urdf (robot description, URDF)
Before this commit: robot box, 1 links, 0 joints
Links:
- link base: geometry collision mesh filename=box.obj scale=1 1 1; visual mesh filename=box.obj scale=1 1 1

File: data/objects/cube/cube.urdf (robot description, URDF)
Before this commit: robot box, 1 links, 0 joints
Links:
- link base: mass .1 -> 10

File: data/objects/tray/tray.urdf (robot description, URDF)
Before this commit: robot tray, 1 links, 0 joints
Links:
- removed link tray_base_link
- added link base_link, mass 1; collision box size=.02 .6 .15; collision box size=.02 .6 .15
