Commit message: 机械臂😍😍😍

File: data/robots/GP12/GP12.urdf (robot description, URDF)
Before this commit: robot motoman_gp12, 8 links, 7 joints
Links:
- link base_link: geometry collision mesh filename=collision/gp12_base_link.stl; visual mesh filename=visual/gp12_base_link.stl
- link link_1_s: geometry collision mesh filename=collision/gp12_link_1_s.stl; visual mesh filename=visual/gp12_link_1_s.stl
- link link_2_l: geometry collision mesh filename=collision/gp12_link_2_l.stl; visual mesh filename=visual/gp12_link_2_l.stl
- link link_3_u: geometry collision mesh filename=collision/gp12_link_3_u.stl; visual mesh filename=visual/gp12_link_3_u.stl
- link link_4_r: geometry collision mesh filename=collision/gp12_link_4_r.stl; visual mesh filename=visual/gp12_link_4_r.stl
- link link_5_b: geometry collision mesh filename=collision/gp12_link_5_b.stl; visual mesh filename=visual/gp12_link_5_b.stl
- link link_6_t: geometry collision mesh filename=collision/gp12_link_6_t.stl; visual mesh filename=visual/gp12_link_6_t.stl

File: data/robots/GP180/GP180.urdf (robot description, URDF)
Before this commit: robot Motoman_GP180, 8 links, 7 joints
Links:
- link Link1: geometry collision mesh filename=Collision/Link1.stl; visual mesh filename=Visual/Link1.stl
- link Link2: geometry collision mesh filename=Collision/Link2.stl; visual mesh filename=Visual/Link2.stl
- link Link3: geometry collision mesh filename=Collision/Link3.stl; visual mesh filename=Visual/Link3.stl
- link Link4: geometry collision mesh filename=Collision/Link4.stl; visual mesh filename=Visual/Link4.stl
- link Link5: geometry collision mesh filename=Collision/Link5.stl; visual mesh filename=Visual/Link5.stl
- link Link6: geometry collision mesh filename=Collision/Link6.stl; visual mesh filename=Visual/Link6.stl
- link base_link: geometry collision mesh filename=Collision/BaseLink.stl; visual mesh filename=Visual/BaseLink.stl

File: data/robots/GP180_120/GP180_120.urdf (robot description, URDF)
Before this commit: robot Motoman_GP180_120, 8 links, 7 joints
Links:
- link Link1: geometry collision mesh filename=Collision/Link1.stl; visual mesh filename=Visual/Link1.stl
- link Link2: geometry collision mesh filename=Collision/Link2.stl; visual mesh filename=Visual/Link2.stl
- link Link3: geometry collision mesh filename=Collision/Link3.stl; visual mesh filename=Visual/Link3.stl
- link Link4: geometry collision mesh filename=Collision/Link4.stl; visual mesh filename=Visual/Link4.stl
- link Link5: geometry collision mesh filename=Collision/Link5.stl; visual mesh filename=Visual/Link5.stl
- link Link6: geometry collision mesh filename=Collision/Link6.stl; visual mesh filename=Visual/Link6.stl
- link base_link: geometry collision mesh filename=Collision/BaseLink.stl; visual mesh filename=Visual/BaseLink.stl

File: data/robots/GP20HL/GP20HL.urdf (robot description, URDF)
Before this commit: robot Motoman_GP20HL, 8 links, 7 joints
Links:
- link Link1: geometry collision mesh filename=Collision/Link1.stl; visual mesh filename=Visual/Link1.stl
- link Link2: geometry collision mesh filename=Collision/Link2.stl; visual mesh filename=Visual/Link2.stl
- link Link3: geometry collision mesh filename=Collision/Link3.stl; visual mesh filename=Visual/Link3.stl
- link Link4: geometry collision mesh filename=Collision/Link4.stl; visual mesh filename=Visual/Link4.stl
- link Link5: geometry collision mesh filename=Collision/Link5.stl; visual mesh filename=Visual/Link5.stl
- link Link6: geometry collision mesh filename=Collision/Link6.stl; visual mesh filename=Visual/Link6.stl
- link base_link: geometry collision mesh filename=Collision/BaseLink.stl; visual mesh filename=Visual/BaseLink.stl

File: data/robots/GP25/GP25.urdf (robot description, URDF)
Before this commit: robot Motoman_GP25, 8 links, 7 joints
Links:
- link Link1: geometry collision mesh filename=Collision/Link1.stl; visual mesh filename=Visual/Link1.stl
- link Link2: geometry collision mesh filename=Collision/Link2.stl; visual mesh filename=Visual/Link2.stl
- link Link3: geometry collision mesh filename=Collision/Link3.stl; visual mesh filename=Visual/Link3.stl
- link Link4: geometry collision mesh filename=Collision/Link4.stl; visual mesh filename=Visual/Link4.stl
- link Link5: geometry collision mesh filename=Collision/Link5.stl; visual mesh filename=Visual/Link5.stl
- link Link6: geometry collision mesh filename=Collision/Link6.stl; visual mesh filename=Visual/Link6.stl
- link base_link: geometry collision mesh filename=Collision/BaseLink.stl; visual mesh filename=Visual/BaseLink.stl

File: data/robots/GP7/GP7.urdf (robot description, URDF)
Before this commit: robot Motoman_GP7, 8 links, 7 joints
Links:
- link Link1: geometry collision mesh filename=Collision/Link1.stl; visual mesh filename=Visual/Link1.stl
- link Link2: geometry collision mesh filename=Collision/Link2.stl; visual mesh filename=Visual/Link2.stl
- link Link3: geometry collision mesh filename=Collision/Link3.stl; visual mesh filename=Visual/Link3.stl
- link Link4: geometry collision mesh filename=Collision/Link4.stl; visual mesh filename=Visual/Link4.stl
- link Link5: geometry collision mesh filename=Collision/Link5.stl; visual mesh filename=Visual/Link5.stl
- link Link6: geometry collision mesh filename=Collision/Link6.stl; visual mesh filename=Visual/Link6.stl
- link base_link: geometry collision mesh filename=Collision/BaseLink.stl; visual mesh filename=Visual/BaseLink.stl

File: data/robots/GP8/GP8.urdf (robot description, URDF)
Before this commit: robot Motoman_GP8, 8 links, 7 joints
Links:
- link Link1: geometry collision mesh filename=Collision/Link1.stl; visual mesh filename=Visual/Link1.stl
- link Link2: geometry collision mesh filename=Collision/Link2.stl; visual mesh filename=Visual/Link2.stl
- link Link3: geometry collision mesh filename=Collision/Link3.stl; visual mesh filename=Visual/Link3.stl
- link Link4: geometry collision mesh filename=Collision/Link4.stl; visual mesh filename=Visual/Link4.stl
- link Link5: geometry collision mesh filename=Collision/Link5.stl; visual mesh filename=Visual/Link5.stl
- link Link6: geometry collision mesh filename=Collision/Link6.stl; visual mesh filename=Visual/Link6.stl
- link base_link: geometry collision mesh filename=Collision/BaseLink.stl; visual mesh filename=Visual/BaseLink.stl

File: data/robots/GP88/GP88.urdf (robot description, URDF)
Before this commit: robot Motoman_GP88, 8 links, 7 joints
Links:
- link Link1: geometry collision mesh filename=Collision/Link1.stl; visual mesh filename=Visual/Link1.stl
- link Link2: geometry collision mesh filename=Collision/Link2.stl; visual mesh filename=Visual/Link2.stl
- link Link3: geometry collision mesh filename=Collision/Link3.stl; visual mesh filename=Visual/Link3.stl
- link Link4: geometry collision mesh filename=Collision/Link4.stl; visual mesh filename=Visual/Link4.stl
- link Link5: geometry collision mesh filename=Collision/Link5.stl; visual mesh filename=Visual/Link5.stl
- link Link6: geometry collision mesh filename=Collision/Link6.stl; visual mesh filename=Visual/Link6.stl
- link base_link: geometry collision mesh filename=Collision/BaseLink.stl; visual mesh filename=Visual/BaseLink.stl

File: data/robots/IRB1200_5_90/IRB1200_5_90.urdf (robot description, URDF)
Before this commit: robot ABB_IRB1200_5_90, 8 links, 7 joints
Links:
- link Link1: geometry collision mesh filename=Collision/Link1.stl; visual mesh filename=Visual/Link1.dae
- link Link2: geometry collision mesh filename=Collision/Link2.stl; visual mesh filename=Visual/Link2.dae
- link Link3: geometry collision mesh filename=Collision/Link3.stl; visual mesh filename=Visual/Link3.dae
- link Link4: geometry collision mesh filename=Collision/Link4.stl; visual mesh filename=Visual/Link4.dae
- link Link5: geometry collision mesh filename=Collision/Link5.stl; visual mesh filename=Visual/Link5.dae
- link Link6: geometry collision mesh filename=Collision/Link6.stl; visual mesh filename=Visual/Link6.dae
- link base_link: geometry collision mesh filename=Collision/BaseLink.stl; visual mesh filename=Visual/BaseLink.dae

File: data/robots/IRB1200_7_70/IRB1200_7_70.urdf (robot description, URDF)
Before this commit: robot ABB_IRB1200_7_70, 8 links, 7 joints
Links:
- link Link1: geometry collision mesh filename=Collision/Link1.stl; visual mesh filename=Visual/Link1.dae
- link Link2: geometry collision mesh filename=Collision/Link2.stl; visual mesh filename=Visual/Link2.dae
- link Link3: geometry collision mesh filename=Collision/Link3.stl; visual mesh filename=Visual/Link3.dae
- link Link4: geometry collision mesh filename=Collision/Link4.stl; visual mesh filename=Visual/Link4.dae
- link Link5: geometry collision mesh filename=Collision/Link5.stl; visual mesh filename=Visual/Link5.dae
- link Link6: geometry collision mesh filename=Collision/Link6.stl; visual mesh filename=Visual/Link6.dae
- link base_link: geometry collision mesh filename=Collision/BaseLink.stl; visual mesh filename=Visual/BaseLink.dae

File: data/robots/IRB1600_6_120/IRB1600_6_120.urdf (robot description, URDF)
Before this commit: robot ABB_IRB1600_6_120, 8 links, 7 joints
Links:
- link Link1: geometry collision mesh filename=Collision/Link1.stl; visual mesh filename=Visual/Link1.stl
- link Link2: geometry collision mesh filename=Collision/Link2.stl; visual mesh filename=Visual/Link2.stl
- link Link3: geometry collision mesh filename=Collision/Link3.stl; visual mesh filename=Visual/Link3.stl
- link Link4: geometry collision mesh filename=Collision/Link4.stl; visual mesh filename=Visual/Link4.stl
- link Link5: geometry collision mesh filename=Collision/Link5.stl; visual mesh filename=Visual/Link5.stl
- link Link6: geometry collision mesh filename=Collision/Link6.stl; visual mesh filename=Visual/Link6.stl
- link base_link: geometry collision mesh filename=Collision/BaseLink.stl; visual mesh filename=Visual/BaseLink.stl

File: data/robots/IRB1600_6_145/IRB1600_10_145.urdf (robot description, URDF)
Before this commit: robot ABB_IRB1600_10_145, 8 links, 7 joints
Links:
- link Link1: geometry collision mesh filename=Collision/Link1.stl; visual mesh filename=Visual/Link1.stl
- link Link2: geometry collision mesh filename=Collision/Link2.stl; visual mesh filename=Visual/Link2.stl
- link Link3: geometry collision mesh filename=Collision/Link3.stl; visual mesh filename=Visual/Link3.stl
- link Link4: geometry collision mesh filename=Collision/Link4.stl; visual mesh filename=Visual/Link4.stl
- link Link5: geometry collision mesh filename=Collision/Link5.stl; visual mesh filename=Visual/Link5.stl
- link Link6: geometry collision mesh filename=Collision/Link6.stl; visual mesh filename=Visual/Link6.stl
- link base_link: geometry collision mesh filename=Collision/BaseLink.stl; visual mesh filename=Visual/BaseLink.stl

File: data/robots/IRB2400_12_155/IRB2400_12_155.urdf (robot description, URDF)
Before this commit: robot ABB_IRB2400_12_155, 10 links, 9 joints
Links:
- link Link1: geometry collision mesh filename=Collision/Link1.stl; visual mesh filename=Visual/Link1.dae
- link Link2: geometry collision mesh filename=Collision/Link2.stl; visual mesh filename=Visual/Link2.dae
- link Link3: geometry collision mesh filename=Collision/Link3.stl; visual mesh filename=Visual/Link3.dae
- link Link4: geometry collision mesh filename=Collision/Link4.stl; visual mesh filename=Visual/Link4.dae
- link Link5: geometry collision mesh filename=Collision/Link5.stl; visual mesh filename=Visual/Link5.dae
- link Link6: geometry collision mesh filename=Collision/Link6.stl; visual mesh filename=Visual/Link6.dae
- link LinkLever_1: geometry collision mesh filename=Collision/LinkLever_1.stl; visual mesh filename=Visual/LinkLever_1.dae
- link LinkLever_2: geometry collision mesh filename=Collision/LinkLever_2.stl; visual mesh filename=Visual/LinkLever_2.dae
- link base_link: geometry collision mesh filename=Collision/BaseLink.stl; visual mesh filename=Visual/BaseLink.dae

File: data/robots/IRB2600_12_165/IRB2600_12_165.urdf (robot description, URDF)
Before this commit: robot ABB_IRB2600_12_165, 8 links, 7 joints
Links:
- link Link1: geometry collision mesh filename=Collision/Link1.stl; visual mesh filename=Visual/Link1.stl
- link Link2: geometry collision mesh filename=Collision/Link2.stl; visual mesh filename=Visual/Link2.stl
- link Link3: geometry collision mesh filename=Collision/Link3.stl; visual mesh filename=Visual/Link3.stl
- link Link4: geometry collision mesh filename=Collision/Link4.stl; visual mesh filename=Visual/Link4.stl
- link Link5: geometry collision mesh filename=Collision/Link5.stl; visual mesh filename=Visual/Link5.stl
- link Link6: geometry collision mesh filename=Collision/Link6.stl; visual mesh filename=Visual/Link6.stl
- link base_link: geometry collision mesh filename=Collision/BaseLink.stl; visual mesh filename=Visual/BaseLink.stl

File: data/robots/IRB2600_12_185/IRB2600_12_185.urdf (robot description, URDF)
Before this commit: robot ABB_IRB2600_12_185, 8 links, 7 joints
Links:
- link Link1: geometry collision mesh filename=Collision/Link1.stl; visual mesh filename=Visual/Link1.stl
- link Link2: geometry collision mesh filename=Collision/Link2.stl; visual mesh filename=Visual/Link2.stl
- link Link3: geometry collision mesh filename=Collision/Link3.stl; visual mesh filename=Visual/Link3.stl
- link Link4: geometry collision mesh filename=Collision/Link4.stl; visual mesh filename=Visual/Link4.stl
- link Link5: geometry collision mesh filename=Collision/Link5.stl; visual mesh filename=Visual/Link5.stl
- link Link6: geometry collision mesh filename=Collision/Link6.stl; visual mesh filename=Visual/Link6.stl
- link base_link: geometry collision mesh filename=Collision/BaseLink.stl; visual mesh filename=Visual/BaseLink.stl

File: data/robots/IRB4400L_30_243/IRB4400L_30_243.urdf (robot description, URDF)
Before this commit: robot ABB_IRB4400L_30_243, 8 links, 7 joints
Links:
- link Link1: geometry collision mesh filename=Collision/Link1.stl; visual mesh filename=Visual/Link1.stl
- link Link2: geometry collision mesh filename=Collision/Link2.stl; visual mesh filename=Visual/Link2.stl
- link Link3: geometry collision mesh filename=Collision/Link3.stl; visual mesh filename=Visual/Link3.stl
- link Link4: geometry collision mesh filename=Collision/Link4.stl; visual mesh filename=Visual/Link4.stl
- link Link5: geometry collision mesh filename=Collision/Link5.stl; visual mesh filename=Visual/Link5.stl
- link Link6: geometry collision mesh filename=Collision/Link6.stl; visual mesh filename=Visual/Link6.stl
- link base_link: geometry collision mesh filename=Collision/BaseLink.stl; visual mesh filename=Visual/BaseLink.stl

File: data/robots/IRB4600_20_250/IRB4600_20_250.urdf (robot description, URDF)
Before this commit: robot ABB_IRB4600_20_250, 8 links, 7 joints
Links:
- link Link1: geometry collision mesh filename=Collision/Link1.stl; visual mesh filename=Visual/Link1.dae
- link Link2: geometry collision mesh filename=Collision/Link2.stl; visual mesh filename=Visual/Link2.dae
- link Link3: geometry collision mesh filename=Collision/Link3.stl; visual mesh filename=Visual/Link3.dae
- link Link4: geometry collision mesh filename=Collision/Link4.stl; visual mesh filename=Visual/Link4.dae
- link Link5: geometry collision mesh filename=Collision/Link5.stl; visual mesh filename=Visual/Link5.dae
- link Link6: geometry collision mesh filename=Collision/Link6.stl; visual mesh filename=Visual/Link6.dae
- link base_link: geometry collision mesh filename=Collision/BaseLink.stl; visual mesh filename=Visual/BaseLink.dae

File: data/robots/IRB4600_40_255/IRB4600_40_255.urdf (robot description, URDF)
Before this commit: robot ABB_IRB4600_40_255, 8 links, 7 joints
Links:
- link Link1: geometry collision mesh filename=Collision/Link1.stl; visual mesh filename=Visual/Link1.dae
- link Link2: geometry collision mesh filename=Collision/Link2.stl; visual mesh filename=Visual/Link2.dae
- link Link3: geometry collision mesh filename=Collision/Link3.stl; visual mesh filename=Visual/Link3.dae
- link Link4: geometry collision mesh filename=Collision/Link4.stl; visual mesh filename=Visual/Link4.dae
- link Link5: geometry collision mesh filename=Collision/Link5.stl; visual mesh filename=Visual/Link5.dae
- link Link6: geometry collision mesh filename=Collision/Link6.stl; visual mesh filename=Visual/Link6.dae
- link base_link: geometry collision mesh filename=Collision/BaseLink.stl; visual mesh filename=Visual/BaseLink.dae

File: data/robots/IRB6700_200_260/IRB6700_200_260.urdf (robot description, URDF)
Before this commit: robot ABB_IRB6700_200_260, 10 links, 9 joints
Links:
- link Link1: geometry collision mesh filename=Collision/Link1.stl; visual mesh filename=Visual/Link1.stl
- link Link2: geometry collision mesh filename=Collision/Link2.stl; visual mesh filename=Visual/Link2.stl
- link Link3: geometry collision mesh filename=Collision/Link3.stl; visual mesh filename=Visual/Link3.stl
- link Link4: geometry collision mesh filename=Collision/Link4.stl; visual mesh filename=Visual/Link4.stl
- link Link5: geometry collision mesh filename=Collision/Link5.stl; visual mesh filename=Visual/Link5.stl
- link Link6: geometry collision mesh filename=Collision/Link6.stl; visual mesh filename=Visual/Link6.stl
- link LinkCylinder: geometry collision mesh filename=Collision/LinkCylinder.stl; visual mesh filename=Visual/LinkCylinder.stl
- link LinkPiston: geometry collision mesh filename=Collision/LinkPiston.stl; visual mesh filename=Visual/LinkPiston.stl
- link base_link: geometry collision mesh filename=Collision/BaseLink.stl; visual mesh filename=Visual/BaseLink.stl

File: data/robots/IRB6700_235_265/IRB6700_235_265.urdf (robot description, URDF)
Before this commit: robot ABB_IRB6700_235_265, 10 links, 9 joints
Links:
- link Link1: geometry collision mesh filename=Collision/Link1.stl; visual mesh filename=Visual/Link1.stl
- link Link2: geometry collision mesh filename=Collision/Link2.stl; visual mesh filename=Visual/Link2.stl
- link Link3: geometry collision mesh filename=Collision/Link3.stl; visual mesh filename=Visual/Link3.stl
- link Link4: geometry collision mesh filename=Collision/Link4.stl; visual mesh filename=Visual/Link4.stl
- link Link5: geometry collision mesh filename=Collision/Link5.stl; visual mesh filename=Visual/Link5.stl
- link Link6: geometry collision mesh filename=Collision/Link6.stl; visual mesh filename=Visual/Link6.stl
- link LinkCylinder: geometry collision mesh filename=Collision/LinkCylinder.stl; visual mesh filename=Visual/LinkCylinder.stl
- link LinkPiston: geometry collision mesh filename=Collision/LinkPiston.stl; visual mesh filename=Visual/LinkPiston.stl
- link base_link: geometry collision mesh filename=Collision/BaseLink.stl; visual mesh filename=Visual/BaseLink.stl
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