Commit message: 阶段提交

File: digitaltwin_data/end_effectors/gripper_gp12/gripper_gp12.urdf (robot description, URDF)
Before this commit: robot universal_robot, 5 links, 4 joints
Joints:
- joint joint_l: limit lower=0.00 upper=0.01 effort=20 velocity=0.2 -> lower=0.00 upper=0.02 effort=20 velocity=0.2; type fixed -> prismatic
- joint joint_r: limit lower=0.00 upper=0.01 effort=20 velocity=0.2 -> lower=0.00 upper=-0.02 effort=20 velocity=0.2; mimic (none) -> joint=joint_l multiplier=1 offset=0; type fixed -> prismatic

File: digitaltwin_data/end_effectors/gripper_ur5/gripper.urdf (robot description, URDF)
Before this commit: robot robotiq_arg2f_85_model, 13 links, 12 joints
Joints:
- joint joint_ee: origin xyz=0.0 0.0 0.14 rpy=3.14 0.0 0.0 -> xyz=0.0 0.0 0.14 rpy=0 0.0 0.0
