Commit message: 基础模型

File: digitaltwin_data/objects/cube/cube.urdf (robot description, URDF)
Before this commit: robot box, 1 links, 0 joints
Links:
- link base: geometry collision box size=1 0.5 0.5; visual box size=1 0.5 0.5

File: digitaltwin_data/objects/cylinder/cylinder.urdf (robot description, URDF)
Before this commit: robot box, 1 links, 0 joints
Links:
- link base: mass 100 -> 1; geometry collision cylinder length=0.5 radius=0.5; visual cylinder length=0.5 radius=0.5

Commit message: 阶段提交

File: digitaltwin_data/objects/cube/cube.urdf (robot description, URDF)
Before this commit: robot box, 1 links, 0 joints
Links:
- link base: geometry collision box size=0.5 0.5 0.7; visual box size=0.5 0.5 0.7
