Commit message: 梅卡曼的垃圾

File: digitaltwin_data/objects/box/box.urdf (robot description, URDF)
Before this commit: robot box, 1 links, 0 joints
Links:
- link base: geometry collision mesh filename=box.urdf.obj scale=1 1 1; visual mesh filename=box.urdf.obj scale=1 1 1

File: digitaltwin_data/objects/cube/cube.urdf (robot description, URDF)
Before this commit: robot box, 1 links, 0 joints
Links:
- link base: geometry collision box size=1 0.5 0.5; visual box size=1 0.5 0.5
